Commit message: Day 3: Upgrade hazardous industrial facility

File: src/hazard_inspection_description/urdf/inspection_robot.urdf.xacro (robot description, xacro)
@@ -22,5 +22,5 @@
         <box size="0.8 0.6 0.25"/>
       </geometry>
-      <origin xyz="0 0 0.25"/>
+      <origin xyz="0 0 0.32"/>
       <material name="robot_gray"/>
     </visual>
@@ -29,9 +29,9 @@
         <box size="0.8 0.6 0.25"/>
       </geometry>
-      <origin xyz="0 0 0.25"/>
+      <origin xyz="0 0 0.32"/>
     </collision>
     <inertial>
       <mass value="10.0"/>
-      <origin xyz="0 0 0.25"/>
+      <origin xyz="0 0 0.32"/>
       <inertia
         ixx="0.75"
@@ -169,5 +169,5 @@
     <parent link="sensor_mast_link"/>
     <child link="lidar_link"/>
-    <origin xyz="0 0 0.25"/>
+    <origin xyz="0 0 0.32"/>
   </joint>
   <!-- ========================= -->

Commit message: Day 4: Finalize robot motion and save facility map

File: src/hazard_inspection_description/urdf/inspection_robot.urdf.xacro (robot description, xacro)
@@ -29,9 +29,9 @@
         <box size="0.8 0.6 0.25"/>
       </geometry>
-      <origin xyz="0 0 0.32"/>
+      <origin xyz="0 0 0.445"/>
     </collision>
     <inertial>
       <mass value="10.0"/>
-      <origin xyz="0 0 0.32"/>
+      <origin xyz="0 0 0.08"/>
       <inertia
         ixx="0.75"
@@ -114,25 +114,66 @@
   </joint>
   <!-- ========================= -->
-  <!-- FRONT CASTER              -->
-  <!-- ========================= -->
-  <link name="front_caster_link">
-    <visual>
-      <geometry>
-        <sphere radius="0.08"/>
-      </geometry>
-      <origin xyz="0 0 0"/>
-      <material name="robot_dark"/>
-    </visual>
-    <collision>
-      <geometry>
-        <sphere radius="0.08"/>
-      </geometry>
-    </collision>
-  </link>
-  <joint name="front_caster_joint"
-         type="fixed">
-    <parent link="base_link"/>
-    <child link="front_caster_link"/>
+  <!-- ========================= -->
+  <!-- PASSIVE SUPPORT WHEELS   -->
+  <!-- ========================= -->
+  <link name="front_support_wheel_link">
+    <visual>
+      <geometry>
+        <cylinder radius="0.08" length="0.06"/>
+      </geometry>
+      <origin xyz="0 0 0" rpy="1.5708 0 0"/>
+      <material name="robot_dark"/>
+    </visual>
+    <inertial>
+      <mass value="0.2"/>
+      <inertia
+        ixx="0.001"
+        ixy="0.0"
+        ixz="0.0"
+        iyy="0.001"
+        iyz="0.0"
+        izz="0.001"/>
+    </inertial>
+  </link>
+  <joint name="front_support_wheel_joint"
+         type="fixed">
+    <parent link="base_link"/>
+    <child link="front_support_wheel_link"/>
     <origin xyz="0.32 0 0.08"/>
+    <axis xyz="0 1 0"/>
+    <dynamics damping="0.05" friction="0.01"/>
+  </joint>
+  <link name="rear_support_wheel_link">
+    <visual>
+      <geometry>
+        <cylinder radius="0.08" length="0.06"/>
+      </geometry>
+      <origin xyz="0 0 0" rpy="1.5708 0 0"/>
+      <material name="robot_dark"/>
+    </visual>
+    <collision>
+      <geometry>
+        <cylinder radius="0.08" length="0.06"/>
+      </geometry>
+      <origin xyz="0 0 0" rpy="1.5708 0 0"/>
+    </collision>
+    <inertial>
+      <mass value="0.2"/>
+      <inertia
+        ixx="0.001"
+        ixy="0.0"
+        ixz="0.0"
+        iyy="0.001"
+        iyz="0.0"
+        izz="0.001"/>
+    </inertial>
+  </link>
+  <joint name="rear_support_wheel_joint"
+         type="fixed">
+    <parent link="base_link"/>
+    <child link="rear_support_wheel_link"/>
+    <origin xyz="-0.32 0 0.08"/>
+    <axis xyz="0 1 0"/>
+    <dynamics damping="0.05" friction="0.01"/>
   </joint>
   <!-- ========================= -->

Commit message: Day 5: Integrate inspection sensors and mission controller

File: src/hazard_inspection_description/urdf/inspection_robot.urdf.xacro (robot description, xacro)
@@ -43,4 +43,100 @@
     </inertial>
   </link>
+  <!-- Temperature Sensor -->
+  <link name="temperature_link">
+    <visual name="temperature_body">
+      <origin xyz="0 0 0"/>
+      <geometry>
+        <cylinder radius="0.045" length="0.16"/>
+      </geometry>
+      <material name="temperature_red">
+        <color rgba="0.8 0.1 0.1 1"/>
+      </material>
+    </visual>
+    <visual name="temperature_probe">
+      <origin xyz="0 0 -0.11"/>
+      <geometry>
+        <cylinder radius="0.018" length="0.08"/>
+      </geometry>
+      <material name="metal">
+        <color rgba="0.65 0.65 0.65 1"/>
+      </material>
+    </visual>
+    <inertial>
+      <mass value="0.05"/>
+      <origin xyz="0 0 0"/>
+      <inertia ixx="0.0001" ixy="0" ixz="0"
+               iyy="0.0001" iyz="0" izz="0.0001"/>
+    </inertial>
+  </link>
+  <joint name="temperature_joint" type="fixed">
+    <parent link="base_link"/>
+    <child link="temperature_link"/>
+    <origin xyz="0.25 0 0.52" rpy="0 0 0"/>
+  </joint>
+  <!-- Gas Sensor -->
+  <link name="gas_sensor_link">
+    <visual name="gas_body">
+      <origin xyz="0 0 0"/>
+      <geometry>
+        <box size="0.14 0.12 0.09"/>
+      </geometry>
+      <material name="gas_yellow">
+        <color rgba="0.9 0.7 0.05 1"/>
+      </material>
+    </visual>
+    <visual name="gas_probe">
+      <origin xyz="0.075 0 0"/>
+      <geometry>
+        <cylinder radius="0.025" length="0.08"/>
+      </geometry>
+      <material name="metal_gas">
+        <color rgba="0.55 0.55 0.55 1"/>
+      </material>
+    </visual>
+    <inertial>
+      <mass value="0.05"/>
+      <origin xyz="0 0 0"/>
+      <inertia ixx="0.0001" ixy="0" ixz="0"
+               iyy="0.0001" iyz="0" izz="0.0001"/>
+    </inertial>
+  </link>
+  <joint name="gas_sensor_joint" type="fixed">
+    <parent link="base_link"/>
+    <child link="gas_sensor_link"/>
+    <origin xyz="0.0 0.25 0.47" rpy="0 0 0"/>
+  </joint>
+  <!-- Pressure Sensor -->
+  <link name="pressure_link">
+    <visual name="pressure_gauge">
+      <origin xyz="0 0 0"/>
+      <geometry>
+        <cylinder radius="0.075" length="0.035"/>
+      </geometry>
+      <material name="pressure_blue">
+        <color rgba="0.1 0.3 0.9 1"/>
+      </material>
+    </visual>
+    <visual name="pressure_connector">
+      <origin xyz="0 0 -0.055"/>
+      <geometry>
+        <cylinder radius="0.025" length="0.08"/>
+      </geometry>
+      <material name="metal_pressure">
+        <color rgba="0.55 0.55 0.55 1"/>
+      </material>
+    </visual>
+    <inertial>
+      <mass value="0.05"/>
+      <origin xyz="0 0 0"/>
+      <inertia ixx="0.0001" ixy="0" ixz="0"
+               iyy="0.0001" iyz="0" izz="0.0001"/>
+    </inertial>
+  </link>
+  <joint name="pressure_joint" type="fixed">
+    <parent link="base_link"/>
+    <child link="pressure_link"/>
+    <origin xyz="-0.25 0 0.52" rpy="0 0 0"/>
+  </joint>
   <!-- ========================= -->
   <!-- LEFT WHEEL                -->
@@ -288,3 +384,13 @@
   </sensor>
 </gazebo>
+  <!-- Gazebo sensor colors -->
+  <gazebo reference="temperature_link">
+    <material>Gazebo/Red</material>
+  </gazebo>
+  <gazebo reference="gas_sensor_link">
+    <material>Gazebo/Yellow</material>
+  </gazebo>
+  <gazebo reference="pressure_link">
+    <material>Gazebo/Blue</material>
+  </gazebo>
 </robot>
